File: eagle_files/soundfield_board_40720_15mm.brd (EAGLE design)
At the start: 15 x 15 mm, 7 parts

Commit message: Board updates
Parts:
- GND_IN: device CM-SparkFun-Connectors:1X01_NO_SILK -> CM-SparkFun-Connectors-2:1X01_2MM
- VDD, VOUT+, VOUT-: device CM-SparkFun-Connectors:1X01_NO_SILK -> CM-SparkFun-Connectors:1X01_2MM
- moved VDD 4.25 mm to (14.8, 9.90)
- moved VOUT+ 2.17 mm to (5.25, 9.95), turned to 270 degrees
- moved C1 1.80 mm to (13.4, 7.35), turned to 270 degrees
- turned GND_IN to 270 degrees
Routing:
- net VDD: track 7.14 -> 5.06 mm
- net VOUT+: track 3.30 -> 4.96 mm
Other:
- board text added: "cmydlarz 2017 Soundfield MEMS mic v0.2"
- board text removed: "cmydlarz 2016 I2S Mic V0.9"
Changed lines of the file:
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@@
 <layer number="17" name="Pads" color="2" fill="1" visible="yes" active="yes"/>
 <layer number="18" name="Vias" color="2" fill="1" visible="yes" active="yes"/>
-<layer number="19" name="Unrouted" color="6" fill="1" visible="no" active="yes"/>
+<layer number="19" name="Unrouted" color="6" fill="1" visible="yes" active="yes"/>
 <layer number="20" name="Dimension" color="15" fill="1" visible="yes" active="yes"/>
 <layer number="21" name="tPlace" color="7" fill="1" visible="yes" active="yes"/>
@@
 <plain>
 <circle x="10" y="10" radius="7.5" width="0.01" layer="20"/>
-<text x="8.25" y="5.2" size="1.27" layer="25">-</text>
-<text x="10.95" y="12.45" size="1.27" layer="25">G</text>
-<text x="11.2" y="3.6" size="1.27" layer="25">Vi</text>
-<text x="5.1" y="9.35" size="1.27" layer="25">+</text>
-<text x="9.9707125" y="8.05" size="0.4064" layer="26" rot="MR0" align="center">cmydlarz 2016
-I2S Mic V0.9</text>
+<text x="7.5" y="5.45" size="1.27" layer="25">-</text>
+<text x="12.35" y="13.5" size="1.27" layer="25">G</text>
+<text x="14.45" y="6.45" size="1.27" layer="25">Vi</text>
+<text x="4.6" y="12.25" size="1.27" layer="25">+</text>
+<text x="10.0207125" y="12" size="0.4064" layer="26" rot="MR0" align="center">cmydlarz 2017
+Soundfield MEMS mic v0.2</text>
 </plain>
 <attributes>
@@
 </autorouter>
 <elements>
-<element name="C1" library="SparkFun-Capacitors" package="0402-CAP" value="" x="14.57" y="8.7" smashed="yes" rot="R90">
-<attribute name="NAME" x="13.8715" y="7.811" size="0.4064" layer="25" rot="R90" display="off"/>
-<attribute name="PROD_ID" value="CAP-12416" x="14.57" y="8.7" size="1.778" layer="27" rot="R90" display="off"/>
-<attribute name="VALUE" x="15.713" y="7.6205" size="0.4064" layer="27" rot="R90"/>
-</element>
-<element name="VOUT-" library="CM-SparkFun-Connectors" package="1X01_NO_SILK" value="" x="10" y="4.95" smashed="yes">
+<element name="C1" library="SparkFun-Capacitors" package="0402-CAP" value="" x="13.38" y="7.35" smashed="yes" rot="R270">
+<attribute name="NAME" x="14.0785" y="8.239" size="0.4064" layer="25" rot="R270" display="off"/>
+<attribute name="PROD_ID" value="CAP-12416" x="13.38" y="7.35" size="1.778" layer="27" rot="R270" display="off"/>
+<attribute name="VALUE" x="12.237" y="8.4295" size="0.4064" layer="27" rot="R270"/>
+</element>
+<element name="VOUT-" library="CM-SparkFun-Connectors" package="1X01_2MM" value="" x="10" y="4.95" smashed="yes">
 <attribute name="VALUE" x="8.73" y="1.775" size="1.27" layer="27"/>
 </element>
-<element name="VOUT+" library="CM-SparkFun-Connectors" package="1X01_NO_SILK" value="" x="6.1" y="7.95" smashed="yes" rot="R180">
-<attribute name="VALUE" x="7.37" y="11.125" size="1.27" layer="27" rot="R180"/>
-</element>
-<element name="VDD" library="CM-SparkFun-Connectors" package="1X01_NO_SILK" value="" x="13" y="6.05" smashed="yes">
-<attribute name="VALUE" x="11.73" y="2.875" size="1.27" layer="27"/>
+<element name="VOUT+" library="CM-SparkFun-Connectors" package="1X01_2MM" value="" x="5.25" y="9.95" smashed="yes" rot="R270">
+<attribute name="VALUE" x="2.075" y="11.22" size="1.27" layer="27" rot="R270"/>
+</element>
+<element name="VDD" library="CM-SparkFun-Connectors" package="1X01_2MM" value="" x="14.8" y="9.9" smashed="yes">
+<attribute name="VALUE" x="13.53" y="6.725" size="1.27" layer="27"/>
 </element>
 <element name="U$1" library="mems_ICS_40720" package=" MEMS_ICS_40720" value=" MEMS_ICS_40720" x="8.5" y="7.32"/>
@@
 <attribute name="VALUE" x="8.73" y="6.825" size="1.27" layer="27"/>
 </element>
-<element name="GND_IN" library="CM-SparkFun-Connectors" package="1X01_NO_SILK" value="" x="9.9" y="14.5" smashed="yes">
-<attribute name="VALUE" x="8.63" y="11.325" size="1.27" layer="27"/>
+<element name="GND_IN" library="CM-SparkFun-Connectors-2" package="1X01_2MM" value="" x="9.9" y="14.5" smashed="yes" rot="R270">
+<attribute name="VALUE" x="6.725" y="15.77" size="1.27" layer="27" rot="R270"/>
 </element>
 </elements>
@@
 <contactref element="U$1" pad="GND"/>
 <contactref element="GND" pad="1"/>
-<via x="14.55" y="10.3" extent="1-16" drill="0.2"/>
 <contactref element="GND_IN" pad="1"/>
-<polygon width="0.4064" layer="16">
+<polygon width="0.4064" layer="16" isolate="0.4064">
 <vertex x="17.3" y="10.05" curve="-90"/>
 <vertex x="9.95" y="2.7"/>
@@
 <vertex x="17.3" y="10.2"/>
 </polygon>
-<wire x1="14.57" y1="9.28" x2="14.55" y2="9.28" width="0.4064" layer="1"/>
-<wire x1="14.55" y1="9.28" x2="14.55" y2="10.3" width="0.4064" layer="1"/>
+<wire x1="13.38" y1="6.77" x2="13.38" y2="5.57" width="0.6096" layer="1"/>
+<wire x1="13.38" y1="5.57" x2="13.4" y2="5.55" width="0.6096" layer="1"/>
+<wire x1="13.4" y1="5.55" x2="13.4" y2="5.45" width="0.6096" layer="1"/>
+<via x="13.4" y="5.45" extent="1-16" drill="0.6" shape="square"/>
 </signal>
 <signal name="VDD">
@@
 <contactref element="VDD" pad="1"/>
 <contactref element="U$1" pad="VDD"/>
-<wire x1="13" y1="6.05" x2="14.57" y2="6.5" width="0.4064" layer="1"/>
-<wire x1="14.57" y1="8.12" x2="14.57" y2="6.5" width="0.4064" layer="1"/>
-<wire x1="10.885" y1="7.915" x2="14.57" y2="7.915" width="0.4064" layer="1"/>
-<wire x1="14.57" y1="7.915" x2="14.57" y2="8.12" width="0.4064" layer="1"/>
+<wire x1="10.885" y1="7.915" x2="13.365" y2="7.915" width="0.6096" layer="1"/>
+<wire x1="13.365" y1="7.915" x2="13.38" y2="7.93" width="0.6096" layer="1"/>
+<wire x1="13.38" y1="7.93" x2="13.38" y2="8.48" width="0.6096" layer="1"/>
+<wire x1="13.38" y1="8.48" x2="14.8" y2="9.9" width="0.6096" layer="1"/>
 </signal>
 <signal name="VOUT+">
@@
 <contactref element="U$1" pad="VOUT+"/>
 <wire x1="8.885" y1="7.915" x2="9.125" y2="7.915" width="0.3048" layer="1"/>
-<wire x1="9.125" y1="7.915" x2="6.1" y2="7.915" width="0.4064" layer="1"/>
-<wire x1="6.1" y1="7.915" x2="6.1" y2="7.95" width="0.4064" layer="1"/>
+<wire x1="9.125" y1="7.915" x2="7.285" y2="7.915" width="0.5" layer="1"/>
+<wire x1="7.285" y1="7.915" x2="5.25" y2="9.95" width="0.5" layer="1"/>
 </signal>
 <signal name="VOUT-">
 <contactref element="VOUT-" pad="1"/>
 <contactref element="U$1" pad="VOUT-"/>
-<wire x1="10.005" y1="7.915" x2="10" y2="7.915" width="0.4064" layer="1"/>
-<wire x1="10" y1="7.915" x2="10" y2="4.95" width="0.4064" layer="1"/>
+<wire x1="10" y1="7.915" x2="10.005" y2="7.915" width="0.4064" layer="1"/>
+<wire x1="10.005" y1="7.915" x2="10.005" y2="4.955" width="0.5" layer="1"/>
+<wire x1="10.005" y1="4.955" x2="10" y2="4.95" width="0.5" layer="1"/>
 </signal>
 <signal name="N$1">
-<polygon width="0.4064" layer="1">
+<polygon width="0.4064" layer="1" isolate="0.4064">
 <vertex x="2.75" y="10" curve="-90"/>
 <vertex x="10" y="17.25"/>
