File: eagle_files/soundfield_board_40720_15mm.sch (EAGLE design)
At the start: 7 parts

Commit message: Board updates
Parts:
- GND_IN: device CM-SparkFun-Connectors:M01PTH_NO_SILK_YES_STOP -> CM-SparkFun-Connectors-2:M01PTH_2MM
- VDD, VOUT+, VOUT-: device CM-SparkFun-Connectors:M01PTH_NO_SILK_YES_STOP -> CM-SparkFun-Connectors:M01PTH_2MM
Changed lines of the file:
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@@
 <part name="GND2" library="supply1" deviceset="GND" device=""/>
 <part name="GND3" library="supply1" deviceset="GND" device=""/>
-<part name="VOUT-" library="CM-SparkFun-Connectors" deviceset="M01" device="PTH_NO_SILK_YES_STOP"/>
-<part name="VOUT+" library="CM-SparkFun-Connectors" deviceset="M01" device="PTH_NO_SILK_YES_STOP"/>
-<part name="VDD" library="CM-SparkFun-Connectors" deviceset="M01" device="PTH_NO_SILK_YES_STOP"/>
+<part name="VOUT-" library="CM-SparkFun-Connectors" deviceset="M01" device="PTH_2MM"/>
+<part name="VOUT+" library="CM-SparkFun-Connectors" deviceset="M01" device="PTH_2MM"/>
+<part name="VDD" library="CM-SparkFun-Connectors" deviceset="M01" device="PTH_2MM"/>
 <part name="GND1" library="supply1" deviceset="GND" device=""/>
 <part name="U$1" library="mems_ICS_40720" deviceset=" MEMS_ICS_40720" device=""/>
 <part name="GND" library="CM-SparkFun-Connectors-large_hole" deviceset="M01" device="PTH_NO_SILK_YES_STOP"/>
-<part name="GND_IN" library="CM-SparkFun-Connectors" deviceset="M01" device="PTH_NO_SILK_YES_STOP"/>
+<part name="GND_IN" library="CM-SparkFun-Connectors-2" deviceset="M01" device="PTH_2MM"/>
 <part name="GND4" library="supply1" deviceset="GND" device=""/>
 </parts>
