File: eagle_files/soundfield_board_40720_12.5mm.brd (EAGLE design)
At the start: 12.5 x 12.5 mm, 7 parts

Commit message: Latest push
Parts:
- GND_IN: device CM-SparkFun-Connectors-2:1X01_2MM -> CM-SparkFun-Connectors-2:1X01
- VDD, VOUT+, VOUT-: device CM-SparkFun-Connectors:1X01_2MM -> CM-SparkFun-Connectors:1X01
Changed lines of the file:
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@@
 <grid distance="0.05" unitdist="mm" unit="mm" style="lines" multiple="2" display="yes" altdistance="0.1" altunitdist="mm" altunit="mm"/>
 <layers>
-<layer number="1" name="Top" color="4" fill="1" visible="no" active="yes"/>
-<layer number="16" name="Bottom" color="1" fill="1" visible="no" active="yes"/>
+<layer number="1" name="Top" color="4" fill="1" visible="yes" active="yes"/>
+<layer number="16" name="Bottom" color="1" fill="1" visible="yes" active="yes"/>
 <layer number="17" name="Pads" color="2" fill="1" visible="yes" active="yes"/>
 <layer number="18" name="Vias" color="2" fill="1" visible="yes" active="yes"/>
@@
 <layer number="20" name="Dimension" color="15" fill="1" visible="yes" active="yes"/>
 <layer number="21" name="tPlace" color="7" fill="1" visible="yes" active="yes"/>
-<layer number="22" name="bPlace" color="7" fill="1" visible="no" active="yes"/>
+<layer number="22" name="bPlace" color="7" fill="1" visible="yes" active="yes"/>
 <layer number="23" name="tOrigins" color="15" fill="1" visible="yes" active="yes"/>
-<layer number="24" name="bOrigins" color="15" fill="1" visible="no" active="yes"/>
+<layer number="24" name="bOrigins" color="15" fill="1" visible="yes" active="yes"/>
 <layer number="25" name="tNames" color="7" fill="1" visible="yes" active="yes"/>
 <layer number="26" name="bNames" color="7" fill="1" visible="yes" active="yes"/>
@@
 <attribute name="VALUE" x="12.237" y="8.4295" size="0.4064" layer="27" rot="R270"/>
 </element>
-<element name="VOUT-" library="CM-SparkFun-Connectors" package="1X01_2MM" value="" x="10" y="5.5" smashed="yes">
+<element name="VOUT-" library="CM-SparkFun-Connectors" package="1X01" value="" x="10" y="5.5" smashed="yes">
 <attribute name="VALUE" x="8.73" y="2.325" size="1.27" layer="27"/>
 </element>
-<element name="VOUT+" library="CM-SparkFun-Connectors" package="1X01_2MM" value="" x="6.25" y="10.1" smashed="yes" rot="R270">
+<element name="VOUT+" library="CM-SparkFun-Connectors" package="1X01" value="" x="6.25" y="10.1" smashed="yes" rot="R270">
 <attribute name="VALUE" x="3.075" y="11.37" size="1.27" layer="27" rot="R270"/>
 </element>
-<element name="VDD" library="CM-SparkFun-Connectors" package="1X01_2MM" value="" x="13.75" y="10" smashed="yes">
+<element name="VDD" library="CM-SparkFun-Connectors" package="1X01" value="" x="13.75" y="10" smashed="yes">
 <attribute name="VALUE" x="12.48" y="6.825" size="1.27" layer="27"/>
 </element>
@@
 <attribute name="VALUE" x="8.73" y="6.825" size="1.27" layer="27"/>
 </element>
-<element name="GND_IN" library="CM-SparkFun-Connectors-2" package="1X01_2MM" value="" x="10.05" y="13.55" smashed="yes" rot="R270">
+<element name="GND_IN" library="CM-SparkFun-Connectors-2" package="1X01" value="" x="10.05" y="13.55" smashed="yes" rot="R270">
 <attribute name="VALUE" x="6.875" y="14.82" size="1.27" layer="27" rot="R270"/>
 </element>
